Commit message: Added next part of the robot arm with link

File: Assets/URDF/BaseFile.urdf (robot description, URDF)
Before this commit: robot simple_robot_arm, 1 links, 0 joints
Links:
- added link link_1, mass 1.0; collision cylinder length=0.5 radius=0.1; visual cylinder length=0.5 radius=0.1
Joints:
- added joint base_to_link1_joint: type revolute, parent base_link, child link_1, origin xyz=0 0 0.1 rpy=0 0 0, axis 0 0 1, limit lower=-1.57 upper=1.57 effort=100.0 velocity=1.0

Commit message: Rigid Body 2

File: Assets/URDF/BaseFile.urdf (robot description, URDF)
Before this commit: robot simple_robot_arm, 2 links, 1 joints
Links:
- added link link_2, mass 1.0; collision cylinder length=0.5 radius=0.1; visual cylinder length=0.5 radius=0.1
Joints:
- added joint link1_to_link2_joint: type revolute, parent link_1, child link_2, origin xyz=0 0 0.25 rpy=0.5 0 0, axis 0 0 1, limit lower=-1.57 upper=1.57 effort=100.0 velocity=1.0
